Commit message: Updated to ROS2

File: urdf/lynxmotion_al5d.urdf.xacro (robot description, xacro)
@@ -8,11 +8,13 @@
         <visual>
             <geometry>
-                <mesh filename="package://lynxmotion_al5d_description/meshes/robot_parts/support.dae" />
-            </geometry>
-            <origin rpy="0 0 0" xyz="0 0 0" />
-        </visual>
-        <collision>
-            <geometry>
-                <mesh filename="package://lynxmotion_al5d_description/meshes/robot_parts/support.dae" />
+                <mesh filename="package://lynxmotion_al5d_description/meshes/visual/support.dae"/>
+            </geometry>
+            <origin rpy="0 0 0" xyz="0 0 0"/>
+        <material name="Silver"/>
+        </visual>
+        <collision>
+            <geometry>
+                <mesh filename="package://lynxmotion_al5d_description/meshes/collision/support.stl"/>
+                <!-- <mesh filename="file:///home/yoha/lynx/lynxmotion_al5d_description/meshes/collision/support.stl"/> -->
             </geometry>
             <origin rpy="0 0 0" xyz="0 0 0" />
@@ -24,11 +26,14 @@
         <visual>
             <geometry>
-                <mesh filename="package://lynxmotion_al5d_description/meshes/robot_parts/rotation_cylinder.dae" />
+                <mesh filename="package://lynxmotion_al5d_description/meshes/visual/rotation_cylinder.dae" />
+                <!-- <mesh filename="file:///home/yoha/lynx/lynxmotion_al5d_description/meshes/visual/rotation_cylinder.dae" /> -->
             </geometry>
             <origin rpy="0 0 0" xyz="0 -0.021 0" />
-        </visual>
-        <collision>
-            <geometry>
-                <mesh filename="package://lynxmotion_al5d_description/meshes/robot_parts/rotation_cylinder.dae" />
+            <material name="Silver"/>
+        </visual>
+        <collision>
+            <geometry>
+                <mesh filename="package://lynxmotion_al5d_description/meshes/collision/rotation_cylinder.stl" />
+                <!-- <mesh filename="file:///home/yoha/lynx/lynxmotion_al5d_description/meshes/collision/rotation_cylinder.stl" /> -->
             </geometry>
             <origin rpy="0 0 0" xyz="0 -0.021 0" />
@@ -40,11 +45,14 @@
         <visual>
             <geometry>
-                <mesh filename="package://lynxmotion_al5d_description/meshes/robot_parts/top_box.dae" />
+                <mesh filename="package://lynxmotion_al5d_description/meshes/visual/top_box.dae" />
+                <!-- <mesh filename="file:///home/yoha/lynx/lynxmotion_al5d_description/meshes/visual/top_box.dae" /> -->
             </geometry>
             <origin xyz="-0.01 0.03 0" rpy="0 0 ${PI}" />
-        </visual>
-        <collision>
-            <geometry>
-                <mesh filename="package://lynxmotion_al5d_description/meshes/robot_parts/top_box.dae" />
+            <material name="BlueGrey"/>
+        </visual>
+        <collision>
+            <geometry>
+                <mesh filename="package://lynxmotion_al5d_description/meshes/collision/top_box.stl" />
+                <!-- <mesh filename="file:///home/yoha/lynx/lynxmotion_al5d_description/meshes/collision/top_box.stl" /> -->
             </geometry>
             <origin xyz="-0.01 0.03 0" rpy="0 0 ${PI}" />
@@ -56,11 +64,15 @@
         <visual>
             <geometry>
-                <mesh filename="package://lynxmotion_al5d_description/meshes/robot_parts/shoulder.dae" />
-            </geometry>
+                <mesh filename="package://lynxmotion_al5d_description/meshes/visual/shoulder.dae" />
+                <!-- <mesh filename="file:///home/yoha/lynx/lynxmotion_al5d_description/meshes/visual/shoulder.dae" /> -->
+            </geometry>
+            <material name="Silver"/>
             <origin rpy="${-5*PI/8} 0 0" xyz="0.005 -0.0625 0.036" />
-        </visual>
-        <collision>
-            <geometry>
-                <mesh filename="package://lynxmotion_al5d_description/meshes/robot_parts/shoulder.dae" />
+            <material name="Silver"/>
+        </visual>
+        <collision>
+            <geometry>
+                <mesh filename="package://lynxmotion_al5d_description/meshes/collision/shoulder.stl" />
+                <!-- <mesh filename="file:///home/yoha/lynx/lynxmotion_al5d_description/meshes/collision/shoulder.stl" /> -->
             </geometry>
             <origin rpy="${-5*PI/8} 0 0" xyz="0.005 -0.0625 0.036" />
@@ -72,11 +84,14 @@
         <visual>
             <geometry>
-                <mesh filename="package://lynxmotion_al5d_description/meshes/robot_parts/elbow.dae" />
+                <mesh filename="package://lynxmotion_al5d_description/meshes/visual/elbow.dae" />
+                <!-- <mesh filename="file:///home/yoha/lynx/lynxmotion_al5d_description/meshes/visual/elbow.dae" /> -->
             </geometry>
             <origin rpy="${-PI-0.895} ${PI} 0" xyz="-0.006 ${tube_length - 2*hs_755eb_depth/5} ${-shoulder_to_elbow - 0.018}" />
-        </visual>
-        <collision>
-            <geometry>
-                <mesh filename="package://lynxmotion_al5d_description/meshes/robot_parts/elbow.dae" />
+            <material name="Silver"/>
+        </visual>
+        <collision>
+            <geometry>
+                <mesh filename="package://lynxmotion_al5d_description/meshes/collision/elbow.stl" />
+                <!-- <mesh filename="file:///home/yoha/lynx/lynxmotion_al5d_description/meshes/collision/elbow.stl" /> -->
             </geometry>
             <origin rpy="${-PI-0.895} ${PI} 0" xyz="-0.005 ${tube_length - 2*hs_755eb_depth/5 + 0.005} ${-shoulder_to_elbow - 0.02} " />
@@ -88,11 +103,14 @@
         <visual>
             <geometry>
-                <mesh filename="package://lynxmotion_al5d_description/meshes/robot_parts/wrist.dae" />
+                <mesh filename="package://lynxmotion_al5d_description/meshes/visual/wrist.dae" />
+                <!-- <mesh filename="file:///home/yoha/lynx/lynxmotion_al5d_description/meshes/visual/wrist.dae" /> -->
             </geometry>
             <origin rpy="${PI} 0 0" xyz="0.005 -0.165 0.0695" />
-        </visual>
-        <collision>
-            <geometry>
-                <mesh filename="package://lynxmotion_al5d_description/meshes/robot_parts/wrist.dae" />
+            <material name="Silver"/>
+        </visual>
+        <collision>
+            <geometry>
+                <mesh filename="package://lynxmotion_al5d_description/meshes/collision/wrist.stl" />
+                <!-- <mesh filename="file:///home/yoha/lynx/lynxmotion_al5d_description/meshes/collision/wrist.stl" /> -->
             </geometry>
             <origin rpy="${PI} 0 0" xyz="0 -0.165 0.067" />
@@ -104,11 +122,14 @@
         <visual>
             <geometry>
-                <mesh filename="package://lynxmotion_al5d_description/meshes/robot_parts/gripper.dae" />
+                <mesh filename="package://lynxmotion_al5d_description/meshes/visual/gripper.dae" />
+                <!-- <mesh filename="file:///home/yoha/lynx/lynxmotion_al5d_description/meshes/visual/gripper.dae" /> -->
             </geometry>
             <origin rpy="${PI/2} 0 ${-PI/2}" xyz="0 -0.02 0.0" />
-        </visual>
-        <collision>
-            <geometry>
-                <mesh filename="package://lynxmotion_al5d_description/meshes/robot_parts/gripper.dae" />
+            <material name="Black"/>
+        </visual>
+        <collision>
+            <geometry>
+                <mesh filename="package://lynxmotion_al5d_description/meshes/collision/gripper.stl" />
+                <!-- <mesh filename="file:///home/yoha/lynx/lynxmotion_al5d_description/meshes/collision/gripper.stl" /> -->
             </geometry>
             <origin rpy="${PI/2} 0 ${-PI/2}" xyz="0 -0.02 0" /> <!---0.021 -0.005" /> -->
@@ -120,11 +141,14 @@
         <visual>
             <geometry>
-                <mesh filename="package://lynxmotion_al5d_description/meshes/robot_parts/finger_left.dae" />
+                <mesh filename="package://lynxmotion_al5d_description/meshes/visual/finger_left.dae" />
+                <!-- <mesh filename="file:///home/yoha/lynx/lynxmotion_al5d_description/meshes/visual/finger_left.dae" /> -->
             </geometry>
             <origin rpy="${PI/2} 0 ${-PI/2}" xyz="0.001 -0.005 0" />
-        </visual>
-        <collision>
-            <geometry>
-                <mesh filename="package://lynxmotion_al5d_description/meshes/robot_parts/finger_left.dae" />
+            <material name="Black"/>
+        </visual>
+        <collision>
+            <geometry>
+                <mesh filename="package://lynxmotion_al5d_description/meshes/collision/finger_left.stl" />
+                <!-- <mesh filename="file:///home/yoha/lynx/lynxmotion_al5d_description/meshes/collision/finger_left.stl" /> -->
             </geometry>
             <origin rpy="${PI/2} 0 ${-PI/2}" xyz="0.001 -0.005 0" />
@@ -136,11 +160,14 @@
         <visual>
             <geometry>
-                <mesh filename="package://lynxmotion_al5d_description/meshes/robot_parts/finger_right.dae" />
+                <mesh filename="package://lynxmotion_al5d_description/meshes/visual/finger_right.dae" />
+                <!-- <mesh filename="file:///home/yoha/lynx/lynxmotion_al5d_description/meshes/visual/finger_right.dae" /> -->
             </geometry>
             <origin rpy="${PI/2} 0 ${-PI/2}" xyz="-0.003 -0.005 0" />
-        </visual>
-        <collision>
-            <geometry>
-                <mesh filename="package://lynxmotion_al5d_description/meshes/robot_parts/finger_right.dae" />
+            <material name="Black"/>
+        </visual>
+        <collision>
+            <geometry>
+                <mesh filename="package://lynxmotion_al5d_description/meshes/collision/finger_right.stl" />
+                <!-- <mesh filename="file:///home/yoha/lynx/lynxmotion_al5d_description/meshes/collision/finger_right.stl" /> -->
             </geometry>
             <origin rpy="${PI/2} 0 ${-PI/2}" xyz="-0.003 -0.005 0" />
@@ -156,5 +183,5 @@
                 <box size="0.01 0.01 0.01" />
             </geometry>
-            <material name="transparent">Gazebo/GreyTransparent</material>
+            <material name="transparent"/>
         </visual>
         <collision>
@@ -173,5 +200,5 @@
             </geometry>
             <origin rpy="0 0 0" xyz="0 0 0" />
-            <material name="transparent">Gazebo/GreyTransparent</material>
+            <material name="transparent"/>
         </visual>
         <collision>
@@ -275,9 +302,62 @@
     <xacro:transmission_block joint_name="Joint5"/>
     <xacro:transmission_block joint_name="Gripper"/>
-    <!-- ros_control plugin -->
+    <!-- ros2_control hardware interface -->
+    <ros2_control name="GazeboSystem" type="system">
+        <hardware>
+            <plugin>gazebo_ros2_control/GazeboSystem</plugin>
+        </hardware>
+        <joint name="Joint1">
+            <command_interface name="position">
+                <param name="min">-3.14159</param>
+                <param name="max">3.14159</param>
+            </command_interface>
+            <state_interface name="position"/>
+            <state_interface name="velocity"/>
+        </joint>
+        <joint name="Joint2">
+            <command_interface name="position">
+                <param name="min">0</param>
+                <param name="max">3.14159</param>
+            </command_interface>
+            <state_interface name="position"/>
+            <state_interface name="velocity"/>
+        </joint>
+        <joint name="Joint3">
+            <command_interface name="position">
+                <param name="min">-3.14159</param>
+                <param name="max">0</param>
+            </command_interface>
+            <state_interface name="position"/>
+            <state_interface name="velocity"/>
+        </joint>
+        <joint name="Joint4">
+            <command_interface name="position">
+                <param name="min">-1.5708</param>
+                <param name="max">1.5708</param>
+            </command_interface>
+            <state_interface name="position"/>
+            <state_interface name="velocity"/>
+        </joint>
+        <joint name="Joint5">
+            <command_interface name="position">
+                <param name="min">-3.14159</param>
+                <param name="max">3.14159</param>
+            </command_interface>
+            <state_interface name="position"/>
+            <state_interface name="velocity"/>
+        </joint>
+        <joint name="Gripper">
+            <command_interface name="position">
+                <param name="min">0</param>
+                <param name="max">0.03175</param>
+            </command_interface>
+            <state_interface name="position"/>
+            <state_interface name="velocity"/>
+        </joint>
+    </ros2_control>
+    <!-- gazebo_ros2_control plugin -->
     <gazebo>
-        <plugin name="gazebo_ros_control" filename="libgazebo_ros_control.so">
-            <robotNamespace>/lynxmotion_al5d</robotNamespace>
-            <legacyModeNS>true</legacyModeNS>
+        <plugin name="gazebo_ros2_control" filename="libgazebo_ros2_control.so">
+            <parameters>$(find lynxmotion_al5d_description)/config/ros2_controllers.yaml</parameters>
         </plugin>
     </gazebo>
@@ -305,11 +385,10 @@
             </camera>
             <plugin filename="libgazebo_ros_camera.so" name="camera_controller">
-                <robotNamespace>/lynxmotion_al5d</robotNamespace>
-                <alwaysOn>true</alwaysOn>
-                <updateRate>1.0</updateRate>
-                <cameraName>external_vision</cameraName>
-                <imageToPIcName>image_raw</imageToPIcName>
-                <cameraInfoToPIcName>camera_info</cameraInfoToPIcName>
-                <frameName>camera_link</frameName>
+                <ros>
+                    <namespace>/lynxmotion_al5d/external_vision</namespace>
+                </ros>
+                <camera_name>external_vision</camera_name>
+                <frame_name>camera_link</frame_name>
+                <hack_baseline>0</hack_baseline>
             </plugin>
         </sensor>

File: urdf/lynxmotion_al5d_properties.urdf.xacro (robot description, xacro)
@@ -2,21 +2,23 @@
 <robot xmlns:xacro="http://www.ros.org/wiki/xacro">
     <!-- Include materials -->
+    <!-- Materials -->
+    <!-- Materials -->
+    <material name="transparent">
+    <color rgba="0.0 0.0 0.0 0.0"/>
+    </material>
     <material name="Black">
-        <color rgba="0.0 0.0 0.0 1.0" />
+    <color rgba="0.0 0.0 0.0 1.0"/>
     </material>
     <material name="Green">
-        <color rgba="0.0 1.0 0.0 1.0" />
+    <color rgba="0.0 1.0 0.0 1.0"/>
     </material>
-    <material name="white">
-        <color rgba="1 1 1 1" />
+    <material name="White">
+    <color rgba="1.0 1.0 1.0 1.0"/>
     </material>
     <material name="Silver">
-        <color rgba="0.8 0.8 0.8 1" />
+    <color rgba="0.8 0.8 0.8 1.0"/>
     </material>
     <material name="BlueGrey">
-        <color rgba="1 87 155 1" />
-    </material>
-    <material name="Transparent">
-        <color rgba="0.0 0.0 0.0 0.0" />
+    <color rgba="0.004 0.341 0.608 1.0"/>
     </material>
     <!-- Setting properties to be used in the program -->
