Commit message: Updates to the lynxarm (not working yet)

File: urdf/lynxmotion_al5d.urdf.xacro (robot description, xacro)
@@ -2,7 +2,5 @@
 <robot name="lynxmotion_al5d" xmlns:xacro="http://www.ros.org/wiki/xacro">
     <xacro:include filename="$(find lynxmotion_al5d_description)/urdf/lynxmotion_al5d_properties.urdf.xacro" />
-    <!-- Base link comprising the board behind the robot and the cylinder at its bottom -->
     <link name="world" />
-    <gazebo reference="world" />
     <link name="robot_support">
         <visual>
@@ -11,10 +9,9 @@
             </geometry>
             <origin rpy="0 0 0" xyz="0 0 0"/>
-        <material name="Silver"/>
+            <material name="Silver"/>
         </visual>
         <collision>
             <geometry>
                 <mesh filename="package://lynxmotion_al5d_description/meshes/collision/support.stl"/>
-                <!-- <mesh filename="file:///home/yoha/lynx/lynxmotion_al5d_description/meshes/collision/support.stl"/> -->
             </geometry>
             <origin rpy="0 0 0" xyz="0 0 0" />
@@ -22,10 +19,8 @@
         <xacro:inertial_matrix mass="${base_mass + board_mass}" ixx="3.6565e-7" ixy="-3.72e-9" ixz="1e-6" iyy="9.404e-8" iyz="4.375e-8" izz="4.1776e-7" xyz="0.000585 0.0602746 0.0170628" />
     </link>
-    <gazebo reference="robot_support" />
     <link name="robot_base_cylinder">
         <visual>
             <geometry>
                 <mesh filename="package://lynxmotion_al5d_description/meshes/visual/rotation_cylinder.dae" />
-                <!-- <mesh filename="file:///home/yoha/lynx/lynxmotion_al5d_description/meshes/visual/rotation_cylinder.dae" /> -->
             </geometry>
             <origin rpy="0 0 0" xyz="0 -0.021 0" />
@@ -35,5 +30,4 @@
             <geometry>
                 <mesh filename="package://lynxmotion_al5d_description/meshes/collision/rotation_cylinder.stl" />
-                <!-- <mesh filename="file:///home/yoha/lynx/lynxmotion_al5d_description/meshes/collision/rotation_cylinder.stl" /> -->
             </geometry>
             <origin rpy="0 0 0" xyz="0 -0.021 0" />
@@ -41,10 +35,8 @@
         <xacro:inertial_matrix_bis mass="0.01" />
     </link>
-    <gazebo reference="robot_base_cylinder" />
     <link name="robot_base_top_box">
         <visual>
             <geometry>
                 <mesh filename="package://lynxmotion_al5d_description/meshes/visual/top_box.dae" />
-                <!-- <mesh filename="file:///home/yoha/lynx/lynxmotion_al5d_description/meshes/visual/top_box.dae" /> -->
             </geometry>
             <origin xyz="-0.01 0.03 0" rpy="0 0 ${PI}" />
@@ -54,5 +46,4 @@
             <geometry>
                 <mesh filename="package://lynxmotion_al5d_description/meshes/collision/top_box.stl" />
-                <!-- <mesh filename="file:///home/yoha/lynx/lynxmotion_al5d_description/meshes/collision/top_box.stl" /> -->
             </geometry>
             <origin xyz="-0.01 0.03 0" rpy="0 0 ${PI}" />
@@ -60,19 +51,15 @@
         <xacro:inertial_matrix_bis mass="${top_box_mass}" />
     </link>
-    <gazebo reference="robot_base_top_box" />
     <link name="shoulder">
         <visual>
             <geometry>
                 <mesh filename="package://lynxmotion_al5d_description/meshes/visual/shoulder.dae" />
-                <!-- <mesh filename="file:///home/yoha/lynx/lynxmotion_al5d_description/meshes/visual/shoulder.dae" /> -->
             </geometry>
             <material name="Silver"/>
             <origin rpy="${-5*PI/8} 0 0" xyz="0.005 -0.0625 0.036" />
-            <material name="Silver"/>
         </visual>
         <collision>
             <geometry>
                 <mesh filename="package://lynxmotion_al5d_description/meshes/collision/shoulder.stl" />
-                <!-- <mesh filename="file:///home/yoha/lynx/lynxmotion_al5d_description/meshes/collision/shoulder.stl" /> -->
             </geometry>
             <origin rpy="${-5*PI/8} 0 0" xyz="0.005 -0.0625 0.036" />
@@ -80,10 +67,8 @@
         <xacro:inertial_matrix_bis mass="${shoulder_mass}" />
     </link>
-    <gazebo reference="shoulder" />
     <link name="elbow">
         <visual>
             <geometry>
                 <mesh filename="package://lynxmotion_al5d_description/meshes/visual/elbow.dae" />
-                <!-- <mesh filename="file:///home/yoha/lynx/lynxmotion_al5d_description/meshes/visual/elbow.dae" /> -->
             </geometry>
             <origin rpy="${-PI-0.895} ${PI} 0" xyz="-0.006 ${tube_length - 2*hs_755eb_depth/5} ${-shoulder_to_elbow - 0.018}" />
@@ -93,16 +78,13 @@
             <geometry>
                 <mesh filename="package://lynxmotion_al5d_description/meshes/collision/elbow.stl" />
-                <!-- <mesh filename="file:///home/yoha/lynx/lynxmotion_al5d_description/meshes/collision/elbow.stl" /> -->
-            </geometry>
-            <origin rpy="${-PI-0.895} ${PI} 0" xyz="-0.005 ${tube_length - 2*hs_755eb_depth/5 + 0.005} ${-shoulder_to_elbow - 0.02} " />
+            </geometry>
+            <origin rpy="${-PI-0.895} ${PI} 0" xyz="-0.005 ${tube_length - 2*hs_755eb_depth/5 + 0.005} ${-shoulder_to_elbow - 0.02}" />
         </collision>
         <xacro:inertial_matrix_bis mass="${hs_755eb_mass + hs_645_mass}" />
     </link>
-    <gazebo reference="elbow" />
     <link name="wrist">
         <visual>
             <geometry>
                 <mesh filename="package://lynxmotion_al5d_description/meshes/visual/wrist.dae" />
-                <!-- <mesh filename="file:///home/yoha/lynx/lynxmotion_al5d_description/meshes/visual/wrist.dae" /> -->
             </geometry>
             <origin rpy="${PI} 0 0" xyz="0.005 -0.165 0.0695" />
@@ -112,5 +94,4 @@
             <geometry>
                 <mesh filename="package://lynxmotion_al5d_description/meshes/collision/wrist.stl" />
-                <!-- <mesh filename="file:///home/yoha/lynx/lynxmotion_al5d_description/meshes/collision/wrist.stl" /> -->
             </geometry>
             <origin rpy="${PI} 0 0" xyz="0 -0.165 0.067" />
@@ -118,10 +99,8 @@
         <xacro:inertial_matrix_bis mass="0.031" />
     </link>
-    <gazebo reference="wrist" />
     <link name="gripper">
         <visual>
             <geometry>
                 <mesh filename="package://lynxmotion_al5d_description/meshes/visual/gripper.dae" />
-                <!-- <mesh filename="file:///home/yoha/lynx/lynxmotion_al5d_description/meshes/visual/gripper.dae" /> -->
             </geometry>
             <origin rpy="${PI/2} 0 ${-PI/2}" xyz="0 -0.02 0.0" />
@@ -131,16 +110,13 @@
             <geometry>
                 <mesh filename="package://lynxmotion_al5d_description/meshes/collision/gripper.stl" />
-                <!-- <mesh filename="file:///home/yoha/lynx/lynxmotion_al5d_description/meshes/collision/gripper.stl" /> -->
-            </geometry>
-            <origin rpy="${PI/2} 0 ${-PI/2}" xyz="0 -0.02 0" /> <!---0.021 -0.005" /> -->
+            </geometry>
+            <origin rpy="${PI/2} 0 ${-PI/2}" xyz="0 -0.02 0" />
         </collision>
         <xacro:inertial_matrix_bis mass="0.042" />
     </link>
-    <gazebo reference="gripper" />
     <link name="left_finger">
         <visual>
             <geometry>
                 <mesh filename="package://lynxmotion_al5d_description/meshes/visual/finger_left.dae" />
-                <!-- <mesh filename="file:///home/yoha/lynx/lynxmotion_al5d_description/meshes/visual/finger_left.dae" /> -->
             </geometry>
             <origin rpy="${PI/2} 0 ${-PI/2}" xyz="0.001 -0.005 0" />
@@ -150,5 +126,4 @@
             <geometry>
                 <mesh filename="package://lynxmotion_al5d_description/meshes/collision/finger_left.stl" />
-                <!-- <mesh filename="file:///home/yoha/lynx/lynxmotion_al5d_description/meshes/collision/finger_left.stl" /> -->
             </geometry>
             <origin rpy="${PI/2} 0 ${-PI/2}" xyz="0.001 -0.005 0" />
@@ -156,10 +131,8 @@
         <xacro:inertial_matrix_bis mass="0.002" />
     </link>
-    <gazebo reference="left_finger" />
     <link name="right_finger">
         <visual>
             <geometry>
                 <mesh filename="package://lynxmotion_al5d_description/meshes/visual/finger_right.dae" />
-                <!-- <mesh filename="file:///home/yoha/lynx/lynxmotion_al5d_description/meshes/visual/finger_right.dae" /> -->
             </geometry>
             <origin rpy="${PI/2} 0 ${-PI/2}" xyz="-0.003 -0.005 0" />
@@ -169,5 +142,4 @@
             <geometry>
                 <mesh filename="package://lynxmotion_al5d_description/meshes/collision/finger_right.stl" />
-                <!-- <mesh filename="file:///home/yoha/lynx/lynxmotion_al5d_description/meshes/collision/finger_right.stl" /> -->
             </geometry>
             <origin rpy="${PI/2} 0 ${-PI/2}" xyz="-0.003 -0.005 0" />
@@ -175,6 +147,4 @@
         <xacro:inertial_matrix_bis mass="0.002" />
     </link>
-    <gazebo reference="right_finger" />
-    <!-- Dummy link used for the gripper -->
     <link name="gripper_mov">
         <visual>
@@ -193,5 +163,4 @@
         <xacro:inertial_matrix_box mass="0.01" width="0.01" height="0.01" depth="0.01" />
     </link>
-    <gazebo reference="gripper_mov" />
     <link name="camera_link">
         <visual>
@@ -210,10 +179,8 @@
         <xacro:inertial_matrix_bis mass="0.0005" />
     </link>
-    <!-- Adding joints -->
     <joint name="world_to_robot" type="fixed">
         <parent link="world" />
         <child link="robot_support" />
         <origin rpy="0 0 ${PI}" />
-        <dynamics damping="1.0" friction="0.8" />
     </joint>
     <joint name="camera_joint" type="fixed">
@@ -222,5 +189,5 @@
         <origin xyz="0 0.17 ${camera_support_depth}" />
     </joint>
-   <joint name="Joint1" type="revolute">
+    <joint name="Joint1" type="revolute">
         <parent link="robot_support" />
         <child link="robot_base_cylinder" />
@@ -233,5 +200,4 @@
         <parent link="robot_base_cylinder" />
         <child link="robot_base_top_box" />
-        <dynamics damping="1.0" friction="0.8" />
     </joint>
     <joint name="Joint2" type="revolute">
@@ -259,5 +225,5 @@
         <dynamics damping="5.0" friction="0.08" />
     </joint>
-   <joint name="Joint5" type="revolute">
+    <joint name="Joint5" type="revolute">
         <parent link="wrist" />
         <child link="gripper" />
@@ -275,5 +241,5 @@
         <dynamics damping="1.0" friction="0.16" />
     </joint>
-   <joint name="left_finger_joint" type="prismatic">
+    <joint name="left_finger_joint" type="prismatic">
         <parent link="gripper" />
         <child link="left_finger" />
@@ -281,26 +247,24 @@
         <axis xyz="-1 0 0" />
         <limit effort="100" velocity="0.1" lower="0" upper="${gripper_base_width/2}" />
-        <!-- Added an offset to fix issues in Rviz -->
         <mimic joint="right_finger_joint" offset="-0.0025" />
         <dynamics damping="1.0" friction="0.16" />
     </joint>
-    <!-- Joint that accept the distance between the two fingers as parameter -->
     <joint name="Gripper" type="prismatic">
         <parent link="gripper" />
         <child link="gripper_mov" />
-        <origin xyz="0.01 0  0" />
+        <origin xyz="0.01 0 0" />
         <limit lower="0" upper="${gripper_base_width}" effort="10" velocity="0.1" />
         <axis xyz="-1 0 0" />
         <dynamics damping="5.0" />
-        <!-- <dynamics friction="0.42" /> -->
-    </joint>
-    <!-- Setting transmissions -->
-    <xacro:transmission_block joint_name="Joint1"/>
-    <xacro:transmission_block joint_name="Joint2"/>
-    <xacro:transmission_block joint_name="Joint3"/>
-    <xacro:transmission_block joint_name="Joint4"/>
-    <xacro:transmission_block joint_name="Joint5"/>
-    <xacro:transmission_block joint_name="Gripper"/>
-    <!-- ros2_control hardware interface -->
+    </joint>
+    <gazebo reference="robot_support"><material>Gazebo/Grey</material></gazebo>
+    <gazebo reference="robot_base_cylinder"><material>Gazebo/Grey</material></gazebo>
+    <gazebo reference="robot_base_top_box"><material>Gazebo/Blue</material></gazebo>
+    <gazebo reference="shoulder"><material>Gazebo/Grey</material></gazebo>
+    <gazebo reference="elbow"><material>Gazebo/Grey</material></gazebo>
+    <gazebo reference="wrist"><material>Gazebo/Grey</material></gazebo>
+    <gazebo reference="gripper"><material>Gazebo/Black</material></gazebo>
+    <gazebo reference="left_finger"><material>Gazebo/Black</material></gazebo>
+    <gazebo reference="right_finger"><material>Gazebo/Black</material></gazebo>
     <ros2_control name="GazeboSystem" type="system">
         <hardware>
@@ -356,5 +320,4 @@
         </joint>
     </ros2_control>
-    <!-- gazebo_ros2_control plugin -->
     <gazebo>
         <plugin name="gazebo_ros2_control" filename="libgazebo_ros2_control.so">
@@ -362,10 +325,10 @@
         </plugin>
     </gazebo>
-    <!-- Setting the mimic joints plugin -->
     <xacro:mimic_joint_plugin_gazebo name_prefix="finger_right"
-    parent_joint="Gripper" mimic_joint="right_finger_joint" multiplier="-0.5"
+        parent_joint="Gripper" mimic_joint="right_finger_joint" multiplier="-0.5"
         has_pid="true" max_effort="10.0" offset="${gripper_base_width/2}" />
     <xacro:mimic_joint_plugin_gazebo name_prefix="finger_left"
-    parent_joint="Gripper" has_pid="true"  mimic_joint="left_finger_joint" multiplier="-0.5" max_effort="10.0" offset="${gripper_base_width/2}" />
+        parent_joint="Gripper" mimic_joint="left_finger_joint" multiplier="-0.5"
+        has_pid="true" max_effort="10.0" offset="${gripper_base_width/2}" />
     <gazebo reference="camera_link">
         <sensor name="external_camera" type="camera">
@@ -390,5 +353,4 @@
                 <camera_name>external_vision</camera_name>
                 <frame_name>camera_link</frame_name>
-                <hack_baseline>0</hack_baseline>
             </plugin>
         </sensor>

File: urdf/lynxmotion_al5d_properties.urdf.xacro (robot description, xacro)
@@ -1,76 +1,28 @@
 <?xml version="1.0" ?>
 <robot xmlns:xacro="http://www.ros.org/wiki/xacro">
-    <!-- Include materials -->
-    <!-- Materials -->
-    <!-- Materials -->
     <material name="transparent">
-    <color rgba="0.0 0.0 0.0 0.0"/>
+        <color rgba="0.0 0.0 0.0 0.0"/>
     </material>
     <material name="Black">
-    <color rgba="0.0 0.0 0.0 1.0"/>
-    </material>
-    <material name="Green">
-    <color rgba="0.0 1.0 0.0 1.0"/>
-    </material>
-    <material name="White">
-    <color rgba="1.0 1.0 1.0 1.0"/>
+        <color rgba="0.0 0.0 0.0 1.0"/>
     </material>
     <material name="Silver">
-    <color rgba="0.8 0.8 0.8 1.0"/>
+        <color rgba="0.8 0.8 0.8 1.0"/>
     </material>
     <material name="BlueGrey">
-    <color rgba="0.004 0.341 0.608 1.0"/>
+        <color rgba="0.004 0.341 0.608 1.0"/>
     </material>
-    <!-- Setting properties to be used in the program -->
-    <xacro:property name="PI" value="3.14159" />
-    <xacro:property name="board_size" value="0.03" />
-    <xacro:property name="board_height" value="0.005" />
-    <xacro:property name="board_mass" value="0.3" />
-    <xacro:property name="base_radius" value="0.025" />
-    <xacro:property name="base_height" value="0.04" />
-    <xacro:property name="base_mass" value="2" />
-    <xacro:property name="top_box_width" value="0.03" />
-    <xacro:property name="top_box_height" value="0.025" />
-    <xacro:property name="top_box_depth" value="0.03" />
-    <xacro:property name="top_box_mass" value="1" />
-    <xacro:property name="shoulder_to_elbow" value="0.146" />
-    <xacro:property name="shoulder_width" value="0.034" />
-    <xacro:property name="shoulder_height" value="0.01"/>
-    <xacro:property name="shoulder_mass" value="0.5" />
-    <xacro:property name="tube_length" value="0.15" />
-    <xacro:property name="tube_radius" value="0.00635" />
-    <xacro:property name="hs_755eb_width" value="0.059" />
-    <xacro:property name="hs_755eb_height" value="0.029" />
-    <xacro:property name="hs_755eb_depth" value="0.05" />
-    <xacro:property name="hs_755eb_mass" value="0.11" />
-    <xacro:property name="hs_645_width" value="0.0406" />
-    <xacro:property name="hs_645_height" value="0.0198" />
-    <xacro:property name="hs_645_depth" value="0.037" />
-    <xacro:property name="hs_645_mass" value="0.05" />
-    <xacro:property name="hs_225_width" value="0.05226" />
-    <xacro:property name="hs_225_height" value="0.01676" />
-    <xacro:property name="hs_225_depth" value="0.032" />
-    <xacro:property name="hs_225_mass" value="0.031" />
-    <xacro:property name="gripper_base_width" value="0.03175" />
-    <xacro:property name="gripper_base_height" value="0.017" />
-    <xacro:property name="gripper_base_depth" value="0.04" />
-    <xacro:property name="finger_width" value="0.003" />
-    <xacro:property name="finger_height" value="0.02" />
-    <xacro:property name="finger_depth" value="0.06" />
-    <xacro:property name="finger_mass" value="0.02" />
-    <xacro:property name="wrist_cylinder_length" value="0.005" />
-    <xacro:property name="wrist_cylinder_radius" value="0.01" />
+    <xacro:property name="PI" value="${pi}" />
+    <xacro:property name="board_mass"         value="0.3" />
+    <xacro:property name="base_mass"           value="2" />
+    <xacro:property name="top_box_mass"        value="1" />
+    <xacro:property name="shoulder_to_elbow"   value="0.146" />
+    <xacro:property name="shoulder_mass"       value="0.5" />
+    <xacro:property name="tube_length"         value="0.15" />
+    <xacro:property name="hs_755eb_depth"      value="0.05" />
+    <xacro:property name="hs_755eb_mass"       value="0.11" />
+    <xacro:property name="hs_645_mass"         value="0.05" />
+    <xacro:property name="gripper_base_width"  value="0.03175" />
     <xacro:property name="camera_support_depth" value="0.25" />
-    <xacro:property name="camera_support_size" value="0.01" />
-    <xacro:property name="camera_support_big_size" value="0.5" />
-    <xacro:property name="camera_support_to_base" value="0.1" />
-    <xacro:property name="camera_support_mass" value="0.2" />
-    <!-- Adding macros for the inertial matrixes -->
-    <xacro:macro name="inertial_matrix_cylinder" params="mass height radius">
-        <inertial>
-            <mass value="${mass}" />
-            <inertia ixx="${(3*radius*radius + height*height)*mass/12}" ixy="0.0" ixz="0.0" iyy="${(3*radius*radius + height*height)*mass/12}" iyz="0.0" izz="${(mass*radius*radius)/2}" />
-        </inertial>
-    </xacro:macro>
     <xacro:macro name="inertial_matrix" params="mass ixx ixy ixz iyy iyz izz xyz">
         <inertial>
@@ -83,42 +35,32 @@
         <inertial>
             <mass value="${mass}" />
-            <inertia ixx="${(depth*depth + height*height)*mass/12}" ixy="0.0" ixz="0.0" iyy="${(width*width + depth*depth)*mass/12}" iyz="0.0" izz="${(width*width + height*height)*mass/12}" />
+            <inertia ixx="${(depth*depth + height*height)*mass/12}" ixy="0.0" ixz="0.0"
+                     iyy="${(width*width + depth*depth)*mass/12}" iyz="0.0"
+                     izz="${(width*width + height*height)*mass/12}" />
         </inertial>
     </xacro:macro>
-   <xacro:macro name="inertial_matrix_bis" params="mass">
-      <inertial>
-        <mass value="${mass}" />
-        <inertia ixx="1.0" ixy="0.0" ixz="0.0" iyy="0.5" iyz="0.0" izz="1.0" />
-      </inertial>
-   </xacro:macro>
-   <!-- Copied from https://github.com/mintar/mimic_joint_gazebo_tutorial/blob/kinetic/urdf/mimic_joint_gazebo_tutorial.urdf.xacro -->
-   <xacro:macro name="mimic_joint_plugin_gazebo" params="name_prefix parent_joint mimic_joint has_pid:=false multiplier:=1.0 offset:=0 sensitiveness:=0.0 max_effort:=1.0 robot_namespace:=''">
-    <gazebo>
-      <plugin name="${name_prefix}mimic_joint_plugin" filename="libroboticsgroup_gazebo_mimic_joint_plugin.so">
-        <joint>${parent_joint}</joint>
-        <mimicJoint>${mimic_joint}</mimicJoint>
-        <xacro:if value="${has_pid}">
-          <hasPID />
-        </xacro:if>
-        <multiplier>${multiplier}</multiplier>
-        <offset>${offset}</offset>
-        <sensitiveness>${sensitiveness}</sensitiveness>
-        <maxEffort>${max_effort}</maxEffort>
-        <xacro:unless value="${robot_namespace == ''}">
-          <robotNamespace>($robot_namespace)</robotNamespace>
-        </xacro:unless>
-      </plugin>
-    </gazebo>
-  </xacro:macro>
-    <xacro:macro name="transmission_block" params="joint_name">
-        <transmission name="tran1">
-            <type>transmission_interface/SimpleTransmission</type>
-            <joint name="${joint_name}">
-                <hardwareInterface>hardware_interface/PositionJointInterface</hardwareInterface>
-            </joint>
-            <actuator name="motor1">
-                <mechanicalReduction>1</mechanicalReduction>
-            </actuator>
-        </transmission>
-   </xacro:macro>
+    <xacro:macro name="inertial_matrix_bis" params="mass">
+        <inertial>
+            <mass value="${mass}" />
+            <inertia ixx="1.0" ixy="0.0" ixz="0.0" iyy="0.5" iyz="0.0" izz="1.0" />
+        </inertial>
+    </xacro:macro>
+    <xacro:macro name="mimic_joint_plugin_gazebo" params="name_prefix parent_joint mimic_joint has_pid:=false multiplier:=1.0 offset:=0 sensitiveness:=0.0 max_effort:=1.0 robot_namespace:=''">
+        <gazebo>
+            <plugin name="${name_prefix}mimic_joint_plugin" filename="libroboticsgroup_upatras_gazebo_mimic_joint_plugin.so">
+                <joint>${parent_joint}</joint>
+                <mimicJoint>${mimic_joint}</mimicJoint>
+                <xacro:if value="${has_pid}">
+                    <hasPID />
+                </xacro:if>
+                <multiplier>${multiplier}</multiplier>
+                <offset>${offset}</offset>
+                <sensitiveness>${sensitiveness}</sensitiveness>
+                <maxEffort>${max_effort}</maxEffort>
+                <xacro:unless value="${robot_namespace == ''}">
+                    <robotNamespace>${robot_namespace}</robotNamespace>
+                </xacro:unless>
+            </plugin>
+        </gazebo>
+    </xacro:macro>
 </robot>
